File: v1.0/rng_rava.brd (EAGLE design)
At the start: 37 x 59.9 mm, 64 parts

Commit message: updating peripherals
Connections:
- net D2: now also MCU.32; no longer MCU.31, MCU.36
- net D3: now also MCU.31; no longer MCU.29
- net D5: now also MCU.29; no longer MCU.25
Routing:
- net D2: track 23.2 -> 15.7 mm, vias 2 -> 1
- net D3: track 20.5 -> 22.0 mm
- net D5: track 23.9 -> 25.2 mm
Changed lines of the file:
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@@
 <drawing>
 <settings>
-<setting alwaysvectorfont="yes"/>
+<setting alwaysvectorfont="no"/>
 <setting verticaltext="up"/>
 </settings>
@@
 <wire x1="16.75" y1="50" x2="9.23" y2="57.52" width="0.254" layer="16"/>
 </signal>
-<signal name="D5">
-<contactref element="MCU" pad="25"/>
-<contactref element="D4,5" pad="2"/>
-<wire x1="23.215" y1="40.14" x2="23.215" y2="41.965" width="0.254" layer="1"/>
-<wire x1="23.215" y1="41.965" x2="23.25" y2="42" width="0.254" layer="1"/>
-<via x="23.25" y="42" extent="1-16" drill="0.35"/>
-<wire x1="23.25" y1="42" x2="23.25" y2="47" width="0.254" layer="16"/>
-<wire x1="23.25" y1="47" x2="19.25" y2="51" width="0.254" layer="16"/>
-<wire x1="19.25" y1="51" x2="17" y2="51" width="0.254" layer="16"/>
-<wire x1="17" y1="51" x2="11.77" y2="56.23" width="0.254" layer="16"/>
-<wire x1="11.77" y1="56.23" x2="11.77" y2="58" width="0.254" layer="16"/>
-</signal>
-<signal name="D2">
-<contactref element="D2" pad="1"/>
-<contactref element="MCU" pad="31"/>
-<wire x1="28.015" y1="40.14" x2="28.015" y2="38.735" width="0.254" layer="1"/>
-<wire x1="28.015" y1="38.735" x2="28.25" y2="38.5" width="0.254" layer="1"/>
-<via x="28.25" y="38.5" extent="1-16" drill="0.35"/>
-<wire x1="28.25" y1="38.5" x2="34.25" y2="38.5" width="0.254" layer="16"/>
-<wire x1="35.75" y1="37" x2="39" y2="37" width="0.254" layer="16"/>
-<wire x1="39" y1="37" x2="40.816" y2="35.184" width="0.254" layer="16"/>
-<wire x1="34.25" y1="38.5" x2="35.75" y2="37" width="0.254" layer="16"/>
-<wire x1="40.816" y1="34.49" x2="40.816" y2="35.184" width="0.254" layer="16"/>
-<contactref element="MCU" pad="36"/>
-<wire x1="31.415" y1="43.54" x2="32.46" y2="43.54" width="0.254" layer="1"/>
-<wire x1="32.873" y1="39.877" x2="34.25" y2="38.5" width="0.254" layer="1"/>
-<wire x1="32.46" y1="43.54" x2="32.873" y2="43.127" width="0.254" layer="1"/>
-<wire x1="32.873" y1="43.127" x2="32.873" y2="39.877" width="0.254" layer="1"/>
-<via x="34.25" y="38.5" extent="1-16" drill="0.35"/>
-</signal>
-<signal name="D3">
-<contactref element="D3" pad="1"/>
-<contactref element="MCU" pad="29"/>
-<wire x1="24.297" y1="36.797" x2="25.75" y2="38.25" width="0.254" layer="16"/>
-<wire x1="11.277" y1="36.797" x2="24.297" y2="36.797" width="0.254" layer="16"/>
-<via x="25.75" y="38.25" extent="1-16" drill="0.35"/>
-<wire x1="8.98" y1="34.5" x2="11.277" y2="36.797" width="0.254" layer="16"/>
-<wire x1="26.415" y1="40.14" x2="26.415" y2="38.915" width="0.254" layer="1"/>
-<wire x1="26.415" y1="38.915" x2="25.75" y2="38.25" width="0.254" layer="1"/>
-</signal>
 <signal name="AVA_Z1">
 <contactref element="R1B" pad="1"/>
@@
 <wire x1="7.758" y1="55.123" x2="7.635" y2="55" width="0.254" layer="1"/>
 </signal>
+<signal name="D2">
+<contactref element="MCU" pad="32"/>
+<contactref element="D2" pad="1"/>
+<wire x1="28.75" y1="38.75" x2="34" y2="38.75" width="0.254" layer="16"/>
+<wire x1="35.75" y1="37" x2="39" y2="37" width="0.254" layer="16"/>
+<wire x1="39" y1="37" x2="40.816" y2="35.184" width="0.254" layer="16"/>
+<wire x1="34" y1="38.75" x2="35.75" y2="37" width="0.254" layer="16"/>
+<wire x1="40.816" y1="34.49" x2="40.816" y2="35.184" width="0.254" layer="16"/>
+<via x="28.75" y="38.75" extent="1-16" drill="0.35"/>
+<wire x1="28.75" y1="38.75" x2="28.688" y2="38.812" width="0.254" layer="1"/>
+<wire x1="28.688" y1="40.013" x2="28.688" y2="38.812" width="0.254" layer="1"/>
+<wire x1="28.688" y1="40.013" x2="28.815" y2="40.14" width="0.254" layer="1"/>
+</signal>
+<signal name="D3">
+<contactref element="MCU" pad="31"/>
+<contactref element="D3" pad="1"/>
+<wire x1="8.98" y1="34.5" x2="11.277" y2="36.797" width="0.254" layer="16"/>
+<wire x1="28.015" y1="40.14" x2="28.015" y2="39.015" width="0.254" layer="1"/>
+<wire x1="28.015" y1="39.015" x2="27" y2="38" width="0.254" layer="1"/>
+<wire x1="27" y1="38" x2="26.25" y2="38" width="0.254" layer="1"/>
+<via x="26.25" y="38" extent="1-16" drill="0.35"/>
+<wire x1="25.047" y1="36.797" x2="26.25" y2="38" width="0.254" layer="16"/>
+<wire x1="11.277" y1="36.797" x2="25.047" y2="36.797" width="0.254" layer="16"/>
+</signal>
+<signal name="D5">
+<contactref element="D4,5" pad="2"/>
+<wire x1="17" y1="51" x2="19.25" y2="51" width="0.254" layer="16"/>
+<wire x1="17" y1="51" x2="11.77" y2="56.23" width="0.254" layer="16"/>
+<wire x1="11.77" y1="56.23" x2="11.77" y2="58" width="0.254" layer="16"/>
+<contactref element="MCU" pad="29"/>
+<wire x1="26.415" y1="40.14" x2="26.415" y2="43.835" width="0.254" layer="1"/>
+<wire x1="26.415" y1="43.835" x2="26.25" y2="44" width="0.254" layer="1"/>
+<via x="26.25" y="44" extent="1-16" drill="0.35"/>
+<wire x1="19.25" y1="51" x2="26.25" y2="44" width="0.254" layer="16"/>
+</signal>
 </signals>
